File: adapter/adapter.kicad_pcb (KiCad board)
At the start: 2 copper layers, 25.4 x 27.4 mm, 2 parts, among them J1 02x07, J2 DIN14

Commit message: initial v2 tweaks
Routing:
- net /5: track 22.6 -> 26.3 mm
- net /7: track 19.6 -> 22.0 mm
- net /3: track 26.2 -> 27.3 mm
- net /1: track 30.8 -> 31.6 mm
- net /9: track 17.6 -> 18.1 mm
