File: idc14-floppy/board.kicad_pcb (KiCad board)
At the start: 2 copper layers, 81.3 x 40.3 mm, 19 parts, among them J1 171826-4, J2 Jack-DC, J3 2x7, J4 02x17, J5 629105150521, SW2 SW_DPDT_x2, U1 L7805

Commit message: 1.10 final
Parts:
- removed C2: 2.2uF, Capacitor_SMD:C_0603_1608Metric
- removed D1, D3: 12v, Diode_SMD:D_0603_1608Metric
- removed J2: Jack-DC, Connector_BarrelJack:BarrelJack_Horizontal
- removed U1: L7805, Package_TO_SOT_SMD:TO-263-2
- D2: value LED -> PWR
- J1: moved to F.Cu
- moved D2 26.1 mm to (118.0, 89.2)
- moved R4 13.0 mm to (123.3, 93.9), turned to 0 degrees
- moved R2 12.5 mm to (121.0, 94.7), turned to -90 degrees
- moved R3 9.77 mm to (123.3, 95.5)
- moved C1 5.30 mm to (124.4, 107.9), turned to 180 degrees
- moved J1 0.65 mm to (121.4, 111.8), turned to 180 degrees
Connections:
- net Net-(R2-Pad2) renamed +3V3
- C1 pad 2: GND -> VSS
- J1 pad 4: +12V -> unconnected-(J1-Pad4)
- J4 pad 1: unconnected-(J4-Pad1) -> GND
- J5 pad 1: Net-(D1-Pad2) -> +5V
Routing:
- net +12V: track 32.1 -> 0.00 mm
- net Net-(D1-Pad2): track 14.3 -> 0.00 mm
- net +5V: track 37.1 -> 25.4 mm
- net Net-(D2-Pad2): track 9.59 -> 6.02 mm
- net +3V3: track 4.26 -> 3.08 mm
- net /FLOPPY_ID1: track 30.7 -> 31.3 mm
Other:
- board text added: "Atari (Drive is set to ID 0) PC (Drive is set to ID 1)"
- board text added: "PWR"
