File: idc14-floppy/board.kicad_pcb (KiCad board)
At the start: 2 copper layers, 81.3 x 40.3 mm, 14 parts, among them J1 171826-4, J3 2x7, J4 02x17, J5 629105150521, SW2 SW_DPDT_x2

Commit message: 1.2 test
Parts:
- added JP1: SW_SPST, Jumper:SolderJumper-2_P1.3mm_Bridged_Pad1.0x1.5mm, F.Cu at (161.8, 101.8)
- added R5: 1k, Resistor_SMD:R_0805_2012Metric, F.Cu at (160.9, 104.9)
- added R6: 1k, Resistor_SMD:R_0805_2012Metric, F.Cu at (160.9, 107.4)
- added R7: 1k, Resistor_SMD:R_0805_2012Metric, F.Cu at (160.9, 110.0)
- added R8: 1k, Resistor_SMD:R_0805_2012Metric, F.Cu at (160.9, 112.5)
- added R9: 1k, Resistor_SMD:R_0805_2012Metric, F.Cu at (160.9, 115.0)
- C1: footprint Capacitor_SMD:C_0603_1608Metric -> Capacitor_SMD:C_0805_2012Metric
- D2: footprint LED_SMD:LED_0603_1608Metric -> LED_SMD:LED_0805_2012Metric
- J3: value 2x7 -> Conn_02x07
- R2, R3, R4: footprint Resistor_SMD:R_0603_1608Metric -> Resistor_SMD:R_0805_2012Metric
- moved R3 0.43 mm to (123.6, 95.8)
- moved R4 0.40 mm to (123.6, 93.7)
- moved C1 0.17 mm to (124.2, 107.9)
Connections:
- net /MOTOR_ON renamed /~{MOTOR_ON}
- net /STEP renamed /~{STEP}
- net /STEP_DIR renamed /~{STEP_DIR}
- net /TRACK_00 renamed /~{TRACK_00}
- net /WRITE_DATA renamed /~{WRITE_DATA}
- net /WRITE_GATE renamed /~{WRITE_GATE}
- J3 pad 14: /WRITE_PROT -> /~{WRITE_PROTECT}
- J4 pad 28: /WRITE_PROT -> /~{WRITE_PROT}
Routing:
- net +5V: track 25.4 -> 81.5 mm, vias 0 -> 1
- net /~{WRITE_PROTECT}: track 0.00 -> 43.8 mm
- net /WRITE_PROT: track 43.8 -> 0.00 mm
- net /~{STEP}: track 29.3 -> 46.0 mm
- net /~{WRITE_GATE}: track 33.5 -> 48.2 mm
- net /~{MOTOR_ON}: track 36.6 -> 49.0 mm
- net Net-(R9-Pad1): track 0.00 -> 12.3 mm
- net /~{WRITE_DATA}: track 29.9 -> 38.4 mm
- net /~{STEP_DIR}: track 26.6 -> 28.4 mm
- net +3V3: track 3.08 -> 3.86 mm
Other:
- board text added: "Atari ST Floppy Adapter v1.2 https://5vsupply.com nick@5vsupply.com"
- board text added: "JP1 Bridged: 1k Shugart Pullups Enabled"
- board text removed: "Atari ST Floppy Adapter v1.1 https://5vsupply.com nick@5vsupply.com"
